Commit message: gazebo starts with joints problems

File: reactor_description/urdf/reactor_description.xacro (robot description, xacro)
@@ -1,8 +1,14 @@
 <?xml version="1.0"?>
-<robot name="reactor_description">
+<robot name="rrbot" xmlns:xacro="http://www.ros.org/wiki/xacro">
   <!-- Import all Gazebo-customization elements, including Gazebo colors -->
   <xacro:include filename="$(find reactor_description)/urdf/reactor.gazebo" />
   <!-- Import Rviz colors -->
   <xacro:include filename="$(find reactor_description)/urdf/materials.xacro" />
+  <!-- Used for fixing robot to Gazebo 'base_link' -->
+  <link name="world"/>
+  <joint name="fixed" type="fixed">
+    <parent link="world"/>
+    <child link="base_link"/>
+  </joint>
   <link
     name="base_link">

Commit message: changes to run gazebo sim

File: reactor_description/urdf/reactor_description.xacro (robot description, xacro)
@@ -1,8 +1,9 @@
 <?xml version="1.0"?>
-<robot name="rrbot" xmlns:xacro="http://www.ros.org/wiki/xacro">
+<robot name="reactor_arm" xmlns:xacro="http://www.ros.org/wiki/xacro">
   <!-- Import all Gazebo-customization elements, including Gazebo colors -->
   <xacro:include filename="$(find reactor_description)/urdf/reactor.gazebo" />
   <!-- Import Rviz colors -->
   <xacro:include filename="$(find reactor_description)/urdf/materials.xacro" />
+  <xacro:property name="PI" value="3.1415926535897931"/>
     <!-- Used for fixing robot to Gazebo 'base_link' -->
   <link name="world"/>
@@ -13,4 +14,12 @@
   <link
     name="base_link">
+    <inertial>
+      <origin xyz="0 0 0" rpy="0 0 0"/>
+      <mass value="1"/>
+      <inertia
+	  ixx="1.0" ixy="0.0" ixz="0.0"
+	  iyy="1.0" iyz="0.0"
+	  izz="1.0"/>
+    </inertial>
     <visual>
       <origin
@@ -153,5 +162,5 @@
       upper="3.141593" />
   </joint>
-  <link
+    <link
     name="forearm_link">
     <inertial>
@@ -211,5 +220,5 @@
       upper="3.141593" />
   </joint>
-  <link
+    <link
     name="wrist_1">
     <inertial>
@@ -269,5 +278,5 @@
       upper="1.57079632679" />
   </joint>
-  <link
+    <link
     name="wrist_2">
     <inertial>
@@ -435,13 +444,3 @@
     </actuator>
   </transmission>
-  <transmission name="gripper_joint_tran">
-    <type>transmission_interface/SimpleTransmission</type>
-    <joint name="gripper_joint">
-      <hardwareInterface>EffortJointInterface</hardwareInterface>
-    </joint>
-    <actuator name="motor6">
-      <hardwareInterface>EffortJointInterface</hardwareInterface>
-      <mechanicalReduction>1</mechanicalReduction>
-    </actuator>
-  </transmission>
 </robot>

Commit message: finally some sensible parameters for robot

File: reactor_description/urdf/reactor_description.xacro (robot description, xacro)
@@ -53,12 +53,9 @@
         rpy="0 0 0" />
       <mass
-        value="0.069055" />
-      <inertia
-        ixx="7.786E-05"
-        ixy="4.5909E-11"
-        ixz="-6.4873E-11"
-        iyy="4.1745E-05"
-        iyz="2.8244E-07"
-        izz="0.0001073" />
+        value="0.2" />
+      <inertia
+	  ixx="0.1" ixy="0.0" ixz="0.0"
+	  iyy="0.1" iyz="0.0"
+	  izz="0.1"/>
     </inertial>
     <visual>
@@ -99,8 +96,8 @@
       xyz="0 0 1" />
     <limit
-      effort="1.5"
-      velocity="6.178465545"
-      lower="-3.141593"
-      upper="3.141593" />
+      effort="10"
+      velocity="6.178465545"
+      lower="-3.1"
+      upper="3.1" />
   </joint>
   <link
@@ -111,12 +108,9 @@
         rpy="0 0 0" />
       <mass
-        value="0.29331" />
-      <inertia
-        ixx="0.00040741"
-        ixy="-1.1578E-09"
-        ixz="-0.00014106"
-        iyy="0.0010604"
-        iyz="1.1578E-09"
-        izz="0.0012838" />
+        value="0.2" />
+      <inertia
+	  ixx="0.1" ixy="0.0" ixz="0.0"
+	  iyy="0.1" iyz="0.0"
+	  izz="0.1"/>
     </inertial>
     <visual>
@@ -157,5 +151,5 @@
       xyz="0 1 0" />
     <limit
-      effort="3.0"
+      effort="15"
       velocity="6.178465545"
       lower="0"
@@ -169,12 +163,9 @@
         rpy="0 0 0" />
       <mass
-        value="0.138705662443181" />
-      <inertia
-        ixx="9.73074886909647E-05"
-        ixy="-2.7259894490049E-06"
-        ixz="8.2757647661483E-07"
-        iyy="0.000291190570207828"
-        iyz="-7.99252279784603E-09"
-        izz="0.000367301178753318" />
+        value="0.2" />
+      <inertia
+	  ixx="0.1" ixy="0.0" ixz="0.0"
+	  iyy="0.1" iyz="0.0"
+	  izz="0.1"/>
     </inertial>
     <visual>
@@ -215,5 +206,5 @@
       xyz="0 -1 0" />
     <limit
-      effort="3.0"
+      effort="20"
       velocity="6.178465545"
       lower="0"
@@ -227,12 +218,9 @@
         rpy="0 0 0" />
       <mass
-        value="0.0605067986491363" />
-      <inertia
-        ixx="1.78648656995261E-05"
-        ixy="1.11621731933541E-10"
-        ixz="3.58888722407994E-06"
-        iyy="2.8352036542644E-05"
-        iyz="-2.18072661043818E-10"
-        izz="2.38673851634115E-05" />
+        value="0.2" />
+      <inertia
+	  ixx="0.1" ixy="0.0" ixz="0.0"
+	  iyy="0.1" iyz="0.0"
+	  izz="0.1"/>
     </inertial>
     <visual>
@@ -273,5 +261,5 @@
       xyz="0 1 0" />
     <limit
-      effort="1.5"
+      effort="10"
       velocity="6.178465545"
       lower="-1.57079632679"
@@ -285,12 +273,9 @@
         rpy="0 0 0" />
       <mass
-        value="0.055706" />
-      <inertia
-        ixx="1.5957E-05"
-        ixy="2.0952E-10"
-        ixz="3.3629E-06"
-        iyy="2.1196E-05"
-        iyz="-2.4643E-10"
-        izz="1.4482E-05" />
+        value="0.2" />
+      <inertia
+	  ixx="0.1" ixy="0.0" ixz="0.0"
+	  iyy="0.1" iyz="0.0"
+	  izz="0.1"/>
     </inertial>
     <visual>
@@ -331,8 +316,8 @@
       xyz="1 0 0" />
     <limit
-      effort="1.5"
-      velocity="6.178465545"
-      lower="-3.141593"
-      upper="3.141593" />
+      effort="10"
+      velocity="6.178465545"
+      lower="-3.1"
+      upper="3.1" />
   </joint>
   <link
@@ -343,12 +328,9 @@
         rpy="0 0 0" />
       <mass
-        value="0.02487" />
-      <inertia
-        ixx="1.5997E-05"
-        ixy="1.6551E-16"
-        ixz="8.3911E-09"
-        iyy="7.3918E-06"
-        iyz="-2.7145E-16"
-        izz="1.5931E-05" />
+        value="0.2" />
+      <inertia
+	  ixx="0.1" ixy="0.0" ixz="0.0"
+	  iyy="0.1" iyz="0.0"
+	  izz="0.1"/>
     </inertial>
     <visual>
@@ -389,8 +371,8 @@
       xyz="1 0 0" />
     <limit
-      effort="1.5"
-      velocity="6.178465545"
-      lower="-3.141593"
-      upper="3.141593" />
+      effort="10"
+      velocity="6.178465545"
+      lower="-3.1"
+      upper="3.1" />
   </joint>
   <transmission name="shoulder_yaw_tran">
